File: ESP32-DEVKIT-S/ESP32-DEVKIT-S-ch340.kicad_pcb (KiCad board)
At the start: 2 copper layers, 28.1 x 43.3 mm, 89 parts, among them J1 JST_2MM_MALE, J2 USB_C_2-LAYER_PADS, J3 Conn_01x20, J4 QWIIC_RIGHT_ANGLE, J5 Conn_01x20, J6 Conn_01x20, J7 QWIIC_RIGHT_ANGLE, Q1 DMG2305UX 20V/4.2A/52mΩ/1.4W, Q2 MBT3904DW1T1, U1 ADXL345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

Commit message: 17.03.23
Parts:
- added >NAME: >VALUE, Silicon-Standard:QFN-10-RSE, B.Cu at (116.0, 65.0)
- added >NAME: >VALUE, Silicon-Standard:QFN-10-RSE, B.Cu at (116.0, 52.5)
- added >NAME: >VALUE, Silicon-Standard:QFN-10-RSE, B.Cu at (116.0, 71.3)
- added >NAME: >VALUE, Silicon-Standard:QFN-10-RSE, B.Cu at (116.0, 58.7)
- added ?: , , F.Cu at (115.7, 71.9)
- added ?: , , F.Cu at (115.7, 65.6)
- added ?: , , F.Cu at (115.7, 53.1)
- moved C10 0.66 mm to (119.4, 58.7), turned to 90 degrees
- moved C9 0.66 mm to (119.4, 65.0), turned to 90 degrees
- moved C8 0.66 mm to (119.4, 71.3), turned to 90 degrees
- moved C11 0.66 mm to (119.4, 52.5), turned to 90 degrees
- moved J7 0.24 mm to (115.8, 47.7)
- moved U6 0.09 mm to (116.0, 65.0)
- moved U8 0.09 mm to (116.0, 52.5)
- moved U5 0.09 mm to (116.0, 71.3)
- moved U7 0.09 mm to (116.0, 58.7)
- moved R10 0.07 mm to (113.0, 70.4)
- moved R11 0.07 mm to (113.0, 69.4)
- moved R12 0.07 mm to (113.0, 68.4)
- moved R13 0.07 mm to (113.0, 67.4)
- moved R14 0.07 mm to (113.0, 65.4)
- moved R15 0.07 mm to (113.0, 64.4)
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Routing:
- net /GPIO_21/SDA: track 112.5 -> 137.7 mm, vias 10 -> 9
- net /A6: track 5.87 -> 29.2 mm
- net /A2: track 8.53 -> 29.5 mm
- net /A10: track 4.57 -> 23.4 mm
- net /A5: track 9.00 -> 24.7 mm
- net /A14: track 15.4 -> 30.6 mm
- net /GPIO_22/SCL: track 111.4 -> 125.8 mm, vias 8 -> 5
- net /A11: track 14.6 -> 25.7 mm
- net /A9: track 6.61 -> 16.9 mm
- net /A8: track 6.68 -> 15.8 mm
- net /A12: track 6.86 -> 14.1 mm
- net GND: track 229.6 -> 236.4 mm, vias 28 -> 32
- net /A7: track 15.8 -> 22.3 mm
- net /A15: track 7.52 -> 13.6 mm
- net /A13: track 6.69 -> 12.4 mm
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
Commit message: 23.04.23
Connections:
- U9 pad 8: /GPIO_1/TX -> /GPIO_3/RX
- U9 pad 9: /GPIO_3/RX -> /GPIO_1/TX
Routing:
- net GND: track 236.4 -> 257.3 mm
- net V_USB: track 36.6 -> 34.0 mm
- net V_BATT: track 45.0 -> 47.4 mm
- net /CH340-DTR: track 9.93 -> 7.69 mm
- net /GPIO_3/RX: track 26.5 -> 28.7 mm
- net Net-(J2-CC2): track 2.97 -> 4.71 mm
- net /D-: track 6.24 -> 6.84 mm
