File: ESP32-DEVKIT-S/ESP32-DEVKIT-S-ch340.kicad_sch (KiCad schematic)
At the start: 76 parts, among them J1 JST_2MM_MALE, J2 USB_C_2-LAYER_PADS, J3 Conn_01x20, J4 QWIIC_RIGHT_ANGLE, J5 Conn_01x20, J6 Conn_01x20, J7 QWIIC_RIGHT_ANGLE, Q1 DMG2305UX 20V/4.2A/52mΩ/1.4W, Q2 MBT3904DW1T1, U1 ADXL345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

Commit message: 23.04.23
Parts:
- removed U$1: SPARKX-LOGO4, SparkFun ESP32 Thing Plus C:SPARKX-MEDIUM, symbol SparkFun ESP32 Thing Plus C-eagle-import:SPARKX-LOGO4
Connections:
- net GPIO_1/TX: no longer U9.8 (TXD)
- net GPIO_3/RX: no longer U9.9 (RXD)
- new net GPIO_1/TX: U9.9 (RXD)
- new net GPIO_3/RX: U9.8 (TXD)
Changed lines of the file:
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@@
     (effects (font (size 0.889 0.889)) (justify left bottom))
   )
-  (label "GPIO_3/RX" (at 320.294 49.53 0) (fields_autoplaced)
+  (label "GPIO_1{slash}TX" (at 320.294 49.53 0) (fields_autoplaced)
     (effects (font (size 0.889 0.889)) (justify left bottom))
   )
@@
     (effects (font (size 0.889 0.889)) (justify right bottom))
   )
-  (label "GPIO_1/TX" (at 320.294 46.99 0) (fields_autoplaced)
+  (label "GPIO_3{slash}RX" (at 320.294 46.99 0) (fields_autoplaced)
     (effects (font (size 0.889 0.889)) (justify left bottom))
   )
@@
         )
       )
-    )
-  )
-  (symbol (lib_id "SparkFun ESP32 Thing Plus C-eagle-import:SPARKX-LOGO4") (at 384.81 251.46 0) (unit 1)
-    (in_bom yes) (on_board no) (dnp no)
-    (property "Reference" "U$1" (at 384.81 251.46 0)
-      (effects (font (size 1.27 1.27)) hide)
-    )
-    (property "Value" "SPARKX-LOGO4" (at 384.81 251.46 0)
-      (effects (font (size 1.27 1.27)) hide)
-    )
-    (property "Footprint" "SparkFun ESP32 Thing Plus C:SPARKX-MEDIUM" (at 384.81 251.46 0)
-      (effects (font (size 1.27 1.27)) hide)
-    )
-    (property "Datasheet" "" (at 384.81 251.46 0)
-      (effects (font (size 1.27 1.27)) hide)
-    )
-    (instances
-      (project "ESP32-DEVKIT-S-ch340"
-        (path "/8468d4d7-80f5-46aa-80f8-c5bed0c248d5"
-          (reference "U$1") (unit 1)
-        )
-      )
