File: ESP32-DEVKIT-S rev1/ESP32-DEVKIT-S/ESP32-DEVKIT-S-ch340.kicad_sch (KiCad schematic)
At the start: 74 parts, among them J1 JST_2MM_MALE, J2 USB_C_2-LAYER_PADS, J3 Conn_01x20, J4 QWIIC_RIGHT_ANGLE, J5 Conn_01x20, J6 Conn_01x20, J7 QWIIC_RIGHT_ANGLE, Q1 DMG2305UX 20V/4.2A/52mΩ/1.4W, Q2 MBT3904DW1T1, U1 ADXL345, U11 MAX17048, U3 >VALUE, U4 MCP73831, U5 ADS1115IDGS, U6 ADS1115IDGS, U7 ADS1115IDGS, U8 ADS1115IDGS, U9 CH340K

Commit message: .
Parts:
- removed S1: Boot, SparkFun ESP32 Thing Plus C:TACTILE_SWITCH_SMD_4.6X2.8MM, symbol SparkFun ESP32 Thing Plus C-eagle-import:MOMENTARY-SWITCH-SPST-SMD-4.6X2.8MM
- removed S2: Reset, SparkFun ESP32 Thing Plus C:TACTILE_SWITCH_SMD_4.6X2.8MM, symbol SparkFun ESP32 Thing Plus C-eagle-import:MOMENTARY-SWITCH-SPST-SMD-4.6X2.8MM
- removed U9: CH340K, Package_SO:SSOP-10_3.9x4.9mm_P1.00mm, symbol Interface_USB:CH340K
- added S1: Boot, Switches:TACTILE_SWITCH_SMD_2.8X1.9MM, symbol Switch:SW_Push_Dual
- added S2: Reset, Switches:TACTILE_SWITCH_SMD_2.8X1.9MM, symbol Switch:SW_Push_Dual
- added U9: CH340C, PCM_Package_SO_AKL:SOIC-16_3.9x9.9mm_P1.27mm, symbol Interface_USB:CH340C
Connections:
- net 3.3V: now also U9.16 (VCC), U9.4 (V3)
- net A1: now also J6.20 (Pin_20); no longer J6.2 (Pin_2)
- net A10: now also J6.9 (Pin_9); no longer J6.13 (Pin_13)
- net A11: now also J6.7 (Pin_7); no longer J6.15 (Pin_15)
- net A12: now also J6.6 (Pin_6); no longer J6.16 (Pin_16)
- net A13: now also J6.5 (Pin_5); no longer J6.17 (Pin_17)
- net A14: now also J6.4 (Pin_4); no longer J6.18 (Pin_18)
- net A15: now also J6.3 (Pin_3); no longer J6.19 (Pin_19)
- net A16: now also J6.2 (Pin_2); no longer J6.20 (Pin_20)
- net A2: now also J6.19 (Pin_19); no longer J6.3 (Pin_3)
- net A3: now also J6.18 (Pin_18); no longer J6.4 (Pin_4)
- net A4: now also J6.17 (Pin_17); no longer J6.5 (Pin_5)
- net A5: now also J6.15 (Pin_15); no longer J6.7 (Pin_7)
- net A6: now also J6.14 (Pin_14); no longer J6.8 (Pin_8)
- net A7: now also J6.13 (Pin_13); no longer J6.9 (Pin_9)
- net A8: now also J6.12 (Pin_12); no longer J6.10 (Pin_10)
- net A9: now also J6.10 (Pin_10); no longer J6.12 (Pin_12)
- net CH340-DTR: now also U9.13 (~{DTR})
- net CH340-RTS: now also U9.14 (~{RTS})
- net D+: now also U9.5 (UD+)
- net D-: now also U9.6 (UD-)
- net GND: now also J6.16 (Pin_16), J6.8 (Pin_8), S1.2, S1.4, S2.2, S2.4, U9.1 (GND); no longer J6.14 (Pin_14), J6.6 (Pin_6)
- net GPIO_0/ADC2_1/QPWR: now also S1.1, S1.3
- net GPIO_1/TX: now also U9.3 (RXD)
- net GPIO_3/RX: now also U9.2 (TXD)
- net ~{RESET}: now also S2.1, S2.3
Other:
- moved on the sheet: C1, C12, C13, C14, C3, C5, D1, D2, D5, J4, J6, JP1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

Commit message: .
Parts:
- added SW1: ON/OFF, Button_Switch_SMD:SW_SPDT_k3-1295, symbol Switch:SW_SPDT
- renumbered R32 to R29, R33 to R30, R34 to R31
Connections:
- net A1: now also J6.19 (Pin_19), U5.7 (AIN3); no longer J6.20 (Pin_20), U5.4 (AIN0)
- net A10: now also J6.8 (Pin_8), U7.6 (AIN2); no longer J6.9 (Pin_9), U7.5 (AIN1)
- net A11: now also J6.6 (Pin_6), U7.5 (AIN1); no longer J6.7 (Pin_7), U7.6 (AIN2)
- net A12: now also J6.5 (Pin_5), U7.4 (AIN0); no longer J6.6 (Pin_6), U7.7 (AIN3)
- net A13: now also J6.4 (Pin_4), U8.7 (AIN3); no longer J6.5 (Pin_5), U8.4 (AIN0)
- net A14: now also J6.3 (Pin_3), U8.6 (AIN2); no longer J6.4 (Pin_4), U8.5 (AIN1)
- net A15: now also J6.2 (Pin_2), U8.5 (AIN1); no longer J6.3 (Pin_3), U8.6 (AIN2)
- net A16: now also J6.1 (Pin_1), U8.4 (AIN0); no longer J6.2 (Pin_2), U8.7 (AIN3)
- net A2: now also J6.18 (Pin_18), U5.6 (AIN2); no longer J6.19 (Pin_19), U5.5 (AIN1)
- net A3: now also J6.17 (Pin_17), U5.5 (AIN1); no longer J6.18 (Pin_18), U5.6 (AIN2)
- net A4: now also J6.16 (Pin_16), U5.4 (AIN0); no longer J6.17 (Pin_17), U5.7 (AIN3)
- net A5: now also J6.14 (Pin_14), U6.7 (AIN3); no longer J6.15 (Pin_15), U6.4 (AIN0)
- net A6: now also J6.13 (Pin_13), U6.6 (AIN2); no longer J6.14 (Pin_14), U6.5 (AIN1)
- net A7: now also J6.12 (Pin_12), U6.5 (AIN1); no longer J6.13 (Pin_13), U6.6 (AIN2)
- net A8: now also J6.11 (Pin_11), U6.4 (AIN0); no longer J6.12 (Pin_12), U6.7 (AIN3)
- net A9: now also J6.9 (Pin_9), U7.7 (AIN3); no longer J6.10 (Pin_10), U7.4 (AIN0)
- net GND: now also J6.15 (Pin_15), J6.7 (Pin_7), SW1.GND; no longer J6.16 (Pin_16), J6.8 (Pin_8)
- net V_BATT: now also SW1.3 (C); no longer J1.2 (+)
- new net V: J1.2 (+), SW1.2 (B)

Commit message: .
Parts:
- removed C13: 0.1uF, SparkFun ESP32 Thing Plus C:0402-TIGHT, symbol SparkFun ESP32 Thing Plus C-eagle-import:0.1UF-0402T-16V-10%
- removed C14: 1.0uF, SparkFun ESP32 Thing Plus C:0402-TIGHT, symbol SparkFun ESP32 Thing Plus C-eagle-import:1.0UF-0402T-16V-10%
- removed D5: BLUE, SparkFun ESP32 Thing Plus C:LED-0603, symbol SparkFun ESP32 Thing Plus C-eagle-import:LED-BLUE0603
- removed J3, J6: Conn_01x20, Connector_FFC-FPC:Molex_200528-0200_1x20-1MP_P1.00mm_Horizontal, symbol Connector_Generic:Conn_01x20
- removed J4, J7: QWIIC_RIGHT_ANGLE, SparkFun ESP32 Thing Plus C:JST04_1MM_RA, symbol SparkFun ESP32 Thing Plus C-eagle-import:QWIIC_CONNECTORJS-1MM
- removed U11: MAX17048, SparkFun ESP32 Thing Plus C:DFN-8, symbol SparkFun ESP32 Thing Plus C-eagle-import:MAX17048DFN8
- added C13: 1.0uF, SparkFun ESP32 Thing Plus C:0402-TIGHT, symbol SparkFun ESP32 Thing Plus C-eagle-import:1.0UF-0402T-16V-10%
- added C14: 0.1uF, SparkFun ESP32 Thing Plus C:0402-TIGHT, symbol SparkFun ESP32 Thing Plus C-eagle-import:0.1UF-0402T-16V-10%
- added D4: BLUE, SparkFun ESP32 Thing Plus C:LED-0603, symbol SparkFun ESP32 Thing Plus C-eagle-import:LED-BLUE0603
- added J3, J6: QWIIC_RIGHT_ANGLE, SparkFun ESP32 Thing Plus C:JST04_1MM_RA, symbol SparkFun ESP32 Thing Plus C-eagle-import:QWIIC_CONNECTORJS-1MM
- added J4, J7: Conn_01x20, Connector_FFC-FPC:Molex_200528-0200_1x20-1MP_P1.00mm_Horizontal, symbol Connector_Generic:Conn_01x20
- added U10: MAX17048, SparkFun ESP32 Thing Plus C:DFN-8, symbol SparkFun ESP32 Thing Plus C-eagle-import:MAX17048DFN8
Connections:
- net 3.3V: now also C13.1, J3.2, J6.2, J7.19 (Pin_19), J7.2 (Pin_2)
- net A1: now also J4.19 (Pin_19)
- net A10: now also J4.8 (Pin_8)
- net A11: now also J4.6 (Pin_6)
- net A12: now also J4.5 (Pin_5)
- net A13: now also J4.4 (Pin_4)
- net A14: now also J4.3 (Pin_3)
- net A15: now also J4.2 (Pin_2)
- net A16: now also J4.1 (Pin_1)
- net A2: now also J4.18 (Pin_18)
- net A3: now also J4.17 (Pin_17)
- net A4: now also J4.16 (Pin_16)
- net A5: now also J4.14 (Pin_14)
- net A6: now also J4.13 (Pin_13)
- net A7: now also J4.12 (Pin_12)
- net A8: now also J4.11 (Pin_11)
- net A9: now also J4.9 (Pin_9)
- net GND: now also C13.2, C14.2, D4.C, J3.1, J4.15 (Pin_15), J4.7 (Pin_7), J6.1, J7.1 (Pin_1), J7.20 (Pin_20), U10.1 (CTG), U10.4 (GND), U10.6 (QSTRT), U10.9 (GND)
- net GPIO_0/ADC2_1/QPWR: now also J7.14 (Pin_14); no longer J5.14 (Pin_14)
- net GPIO_1/TX: now also J7.5 (Pin_5); no longer J5.5 (Pin_5)
- net GPIO_10/SWP: now also J5.5 (Pin_5)
- net GPIO_11/SCS: now also J5.4 (Pin_4)
- net GPIO_12/ADC2_5: now also J5.8 (Pin_8)
- net GPIO_13/ADC2_4/LED: now also J5.7 (Pin_7)
- net GPIO_14/ADC2_6: now also J5.9 (Pin_9)
- net GPIO_15/ADC2_3: now also J7.16 (Pin_16); no longer J5.16 (Pin_16)
- net GPIO_16/RX: now also J7.12 (Pin_12); no longer J5.12 (Pin_12)
- net GPIO_17/TX: now also J7.11 (Pin_11); no longer J5.11 (Pin_11)
- net GPIO_18/SCK: now also J7.9 (Pin_9); no longer J5.9 (Pin_9)
- net GPIO_19/CIPO: now also J7.8 (Pin_8); no longer J5.8 (Pin_8)
- net GPIO_2/ADC2_2: now also J7.15 (Pin_15); no longer J5.15 (Pin_15)
- net GPIO_21/SDA: now also J3.3, J6.3, J7.7 (Pin_7), U10.8 (SDA); no longer J5.7 (Pin_7)
- net GPIO_22/SCL: now also J3.4, J6.4, J7.4 (Pin_4), U10.7 (SCL); no longer J5.4 (Pin_4)
- net GPIO_23/COPI: now also J7.3 (Pin_3); no longer J5.3 (Pin_3)
- net GPIO_25/ADC2_8: now also J5.12 (Pin_12)
- net GPIO_26/ADC2_9: now also J5.11 (Pin_11)
- net GPIO_27/ADC2_7: now also J5.10 (Pin_10)
- net GPIO_3/RX: now also J7.6 (Pin_6); no longer J5.6 (Pin_6)
- net GPIO_32/ADC1_4: now also J5.14 (Pin_14)
- net GPIO_33/ADC1_5: now also J5.13 (Pin_13)
- net GPIO_34/ADC1_6: now also J5.16 (Pin_16)
- net GPIO_35/ADC1_7: now also J5.15 (Pin_15)
- net GPIO_36/ADC1_0: now also J5.18 (Pin_18)
- net GPIO_39/ADC1_3: now also J5.17 (Pin_17)
- net GPIO_4/ADC2_0: now also J7.13 (Pin_13); no longer J5.13 (Pin_13)
- net GPIO_5/SD_CS: now also J7.10 (Pin_10); no longer J5.10 (Pin_10)
- net GPIO_6/SCK: now also J5.3 (Pin_3)
- net GPIO_7/SDO: now also J7.18 (Pin_18); no longer J5.18 (Pin_18)
- net GPIO_8/SDI: now also J7.17 (Pin_17); no longer J5.17 (Pin_17)
- net GPIO_9/SHD: now also J5.6 (Pin_6)
- net V_BATT: now also C14.1, U10.2 (CELL), U10.3 (VDD)
- net at R31.2: now also D4.A
