File: ESP32-DEVKIT-S rev1/ESP32-DEVKIT-S-mirror/ESP32-DEVKIT-S-ch340-mirror.kicad_pcb (KiCad board)
At the start: 2 copper layers, 28.9 x 42.5 mm, 94 parts, among them J1 JST_2MM_MALE, J2 USB_C_2-LAYER_PADS, J3 Conn_01x20, J4 QWIIC_RIGHT_ANGLE, J5 Conn_01x20, J6 Conn_01x20, J7 QWIIC_RIGHT_ANGLE, Q1 DMG2305UX 20V/4.2A/52mΩ/1.4W, Q2 MBT3904DW1T1, U1 ADXL345, U11 MAX17048, U3 >VALUE, U4 MCP73831, U5 ADS1115IDGS, U6 ADS1115IDGS, U7 ADS1115IDGS, U8 ADS1115IDGS, U9 CH340K

Commit message: .
Parts:
- removed the >NAME at (107.6, 73.8)
- removed the >NAME at (107.6, 70.8)
- C14, R26, U11: moved to B.Cu
- S1, S2: footprint SparkFun ESP32 Thing Plus C:TACTILE_SWITCH_SMD_4.6X2.8MM -> Switches:TACTILE_SWITCH_SMD_2.8X1.9MM
- U9: value CH340K -> CH340C; footprint Package_SO:SSOP-10_3.9x4.9mm_P1.00mm -> PCM_Package_SO_AKL:SOIC-16_3.9x9.9mm_P1.27mm
- moved R26 5.10 mm to (99.3, 70.2)
- moved C14 3.87 mm to (100.5, 70.6), turned to -90 degrees
- moved C2 2.98 mm to (102.3, 70.6), turned to -90 degrees
- moved U11 2.78 mm to (109.2, 78.6), turned to 180 degrees
- moved C4 2.47 mm to (101.4, 70.6), turned to -90 degrees
- moved S1 1.88 mm to (109.3, 74.6), turned to -90 degrees
- moved U9 1.75 mm to (102.9, 73.1)
- moved S2 1.72 mm to (109.3, 70.9), turned to -90 degrees
- moved C12 1.38 mm to (97.1, 71.3), turned to 90 degrees
- moved Q2 1.13 mm to (101.7, 73.2)
- moved R8 1.07 mm to (100.0, 74.6)
- moved R7 0.72 mm to (103.3, 74.7)
Connections:
- S1 pad 2: /GPIO_0/ADC2_1/QPWR -> GND
- S1 pad 3: GND -> /GPIO_0/ADC2_1/QPWR
- S2 pad 2: /~{RESET} -> GND
- S2 pad 3: GND -> /~{RESET}
- U9 pad 1: /D+ -> GND
- U9 pad 10: 3.3V -> unconnected-(U9-~{DSR}-Pad10)
- U9 pad 2: /D- -> /GPIO_3/RX
- U9 pad 3: GND -> /GPIO_1/TX
- U9 pad 4: /CH340-DTR -> 3.3V
- U9 pad 5: unconnected-(U9-~{CTS}-Pad5) -> /D+
- U9 pad 6: /CH340-RTS -> /D-
- U9 pad 7: 3.3V -> unconnected-(U9-NC-Pad7)
- U9 pad 8: /GPIO_3/RX -> unconnected-(U9-NC-Pad8)
- U9 pad 9: /GPIO_1/TX -> unconnected-(U9-~{CTS}-Pad9)
Routing:
- net 3.3V: track 241.4 -> 258.4 mm
- net /~{RESET}: track 45.3 -> 56.2 mm
- net GND: track 332.3 -> 323.8 mm, vias 96 -> 90
- net /GPIO_21/SDA: track 115.0 -> 121.8 mm
- net /GPIO_22/SCL: track 108.1 -> 114.8 mm, vias 5 -> 7
- net /D-: track 5.03 -> 10.7 mm
- net /D+: track 9.13 -> 5.94 mm
- net /GPIO_8/SDI: track 1.66 -> 4.71 mm
- net V_USB: track 44.2 -> 47.3 mm
- net /CH340-DTR: track 2.15 -> 4.92 mm
- net /GPIO_7/SDO: track 3.21 -> 5.81 mm
- net /GPIO_3/RX: track 28.1 -> 30.2 mm
- net /GPIO_0/ADC2_1/QPWR: track 26.2 -> 28.2 mm, vias 3 -> 1
- net Net-(J2-CC2): track 4.77 -> 6.22 mm
- net /GPIO_2/ADC2_2: track 4.01 -> 2.64 mm
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
Commit message: .
Parts:
- removed the >NAME at (116.0, 65.0)
- removed the >NAME at (116.0, 52.5)
- removed the >NAME at (116.0, 71.3)
- removed the >NAME at (116.0, 58.7)
- removed the ? at (115.7, 71.9)
- removed the ? at (115.7, 65.6)
- removed the ? at (115.7, 53.1)
- removed C1, C10, C11, C14, C2, C3, C8, C9: 1.0uF, SparkFun ESP32 Thing Plus C:0402-TIGHT
- removed C12, C13: 0.1uF, SparkFun ESP32 Thing Plus C:0402-TIGHT
- removed C4, C5: 10uF, SparkFun ESP32 Thing Plus C:0402-TIGHT
- removed C6, C7: 4.7uF, SparkFun ESP32 Thing Plus C:0402-TIGHT
- removed D1: S4 3A/10V/280mV, SparkFun ESP32 Thing Plus C:SOD-323
- removed D2: RED, SparkFun ESP32 Thing Plus C:LED-0603
- removed D3: Yellow, SparkFun ESP32 Thing Plus C:LED-0603
- removed J1: JST_2MM_MALE, SparkFun ESP32 Thing Plus C:JST-2-SMD
- removed J2: USB_C_2-LAYER_PADS, SparkFun ESP32 Thing Plus C:USB-C-16P-2LAYER-PADS
- removed J3, J5, J6: Conn_01x20, Connector_FFC-FPC:Molex_200528-0200_1x20-1MP_P1.00mm_Horizontal
- removed J4, J7: QWIIC_RIGHT_ANGLE, SparkFun ESP32 Thing Plus C:JST04_1MM_RA
- removed Q1: DMG2305UX 20V/4.2A/52mΩ/1.4W, SparkFun ESP32 Thing Plus C:SOT23-3
- removed Q2: MBT3904DW1T1, SparkFun ESP32 Thing Plus C:SC70-6
- removed R1, R26, R3, R4, R7, R8: 10k, SparkFun ESP32 Thing Plus C:0402-TIGHT
- removed R10, R11, R12, R13, R14, R15, R16, R17, R18, R19, R20, R21, R22, R23, R24, R25: 150k, SparkFun ESP32 Thing Plus C:0402-TIGHT
- removed R2, R5, R6: 4k7, SparkFun ESP32 Thing Plus C:0402-TIGHT
- removed R27, R9: 1k, SparkFun ESP32 Thing Plus C:0402-TIGHT
- removed R28: 2.0k, SparkFun ESP32 Thing Plus C:0402-TIGHT
- removed S1: Boot, Switches:TACTILE_SWITCH_SMD_2.8X1.9MM
- removed S2: Reset, Switches:TACTILE_SWITCH_SMD_2.8X1.9MM
- removed U1: ADXL345, Package_LGA:LGA-14_3x5mm_P0.8mm_LayoutBorder1x6y
- removed U2: , SparkFun ESP32 Thing Plus C:SOT23-5
- removed U3: >VALUE, SparkFun ESP32 Thing Plus C:ESP-WROOM-32-NARROW
- removed U4: MCP73831, SparkFun ESP32 Thing Plus C:SOT23-5
- removed U5, U6, U7, U8: ADS1115IDGS, Package_SO:TSSOP-10_3x3mm_P0.5mm
- removed U9: CH340C, PCM_Package_SO_AKL:SOIC-16_3.9x9.9mm_P1.27mm
- added >NAME: >VALUE, Silicon-Standard:QFN-10-RSE, B.Cu at (117.4, 53.0)
- added >NAME: >VALUE, Silicon-Standard:QFN-10-RSE, B.Cu at (117.4, 71.9)
- added >NAME: >VALUE, Silicon-Standard:QFN-10-RSE, B.Cu at (117.4, 59.3)
- added >NAME: >VALUE, Silicon-Standard:QFN-10-RSE, B.Cu at (117.4, 65.6)
- added C15: 1.0uF, SparkFun ESP32 Thing Plus C:0402-TIGHT, B.Cu at (101.9, 77.0)
- added C16: 1.0uF, SparkFun ESP32 Thing Plus C:0402-TIGHT, B.Cu at (102.3, 70.6)
- added C17: 1.0uF, SparkFun ESP32 Thing Plus C:0402-TIGHT, B.Cu at (101.6, 54.3)
- added C18: 10uF, SparkFun ESP32 Thing Plus C:0402-TIGHT, B.Cu at (101.4, 70.6)
- added C19: 10uF, SparkFun ESP32 Thing Plus C:0402-TIGHT, B.Cu at (100.7, 54.3)
- added C20: 4.7uF, SparkFun ESP32 Thing Plus C:0402-TIGHT, B.Cu at (102.3, 78.4)
- added C21: 4.7uF, SparkFun ESP32 Thing Plus C:0402-TIGHT, F.Cu at (109.4, 81.7)
- added C22: 1.0uF, SparkFun ESP32 Thing Plus C:0402-TIGHT, B.Cu at (113.5, 74.4)
- added C23: 1.0uF, SparkFun ESP32 Thing Plus C:0402-TIGHT, B.Cu at (113.5, 73.5)
- added C24: 1.0uF, SparkFun ESP32 Thing Plus C:0402-TIGHT, B.Cu at (113.5, 72.6)
- added C25: 1.0uF, SparkFun ESP32 Thing Plus C:0402-TIGHT, B.Cu at (113.5, 71.7)
- added C26: 0.1uF, SparkFun ESP32 Thing Plus C:0402-TIGHT, F.Cu at (97.1, 71.3)
- added C27: 1.0uF, SparkFun ESP32 Thing Plus C:0402-TIGHT, B.Cu at (100.5, 70.6)
- added C28: 0.1uF, SparkFun ESP32 Thing Plus C:0402-TIGHT, B.Cu at (105.8, 81.0)
- added D6: RED, SparkFun ESP32 Thing Plus C:LED-0603, F.Cu at (95.6, 83.7)
- added D7: Yellow, SparkFun ESP32 Thing Plus C:LED-0603, F.Cu at (106.7, 83.7)
- added D8: BLUE, SparkFun ESP32 Thing Plus C:LED-0603, F.Cu at (93.4, 70.1)
- added J10: QWIIC_RIGHT_ANGLE, SparkFun ESP32 Thing Plus C:JST04_1MM_RA, F.Cu at (115.9, 47.7)
- added J11: Conn_01x20, Connector_FFC-FPC:Molex_200528-0200_1x20-1MP_P1.00mm_Horizontal, F.Cu at (114.5, 61.9)
- added J12: Conn_01x20, Connector_FFC-FPC:Molex_200528-0200_1x20-1MP_P1.00mm_Horizontal, B.Cu at (96.6, 63.3)
- added J13: QWIIC_RIGHT_ANGLE, SparkFun ESP32 Thing Plus C:JST04_1MM_RA, F.Cu at (96.7, 74.3)
- added J14: Conn_01x20, Connector_FFC-FPC:Molex_200528-0200_1x20-1MP_P1.00mm_Horizontal, B.Cu at (105.7, 63.3)
- added J8: JST_2MM_MALE, SparkFun ESP32 Thing Plus C:JST-2-SMD, F.Cu at (117.3, 80.9)
- added J9: USB_C_2-LAYER_PADS, SparkFun ESP32 Thing Plus C:USB-C-16P-2LAYER-PADS, F.Cu at (101.1, 77.6)
- added Q3: DMG2305UX 20V/4.2A/52mΩ/1.4W, SparkFun ESP32 Thing Plus C:SOT23-3, B.Cu at (103.1, 80.9)
- added Q4: MBT3904DW1T1, SparkFun ESP32 Thing Plus C:SC70-6, B.Cu at (101.4, 73.0)
- added R35: 10k, SparkFun ESP32 Thing Plus C:0402-TIGHT, B.Cu at (100.1, 67.6)
- added R36: 4k7, SparkFun ESP32 Thing Plus C:0402-TIGHT, B.Cu at (103.3, 58.8)
- added R37: 4k7, SparkFun ESP32 Thing Plus C:0402-TIGHT, B.Cu at (103.3, 60.7)
- added R38: 10k, SparkFun ESP32 Thing Plus C:0402-TIGHT, B.Cu at (103.1, 74.1)
- added R39: 10k, SparkFun ESP32 Thing Plus C:0402-TIGHT, B.Cu at (99.7, 73.7)
- added R40: 1k, SparkFun ESP32 Thing Plus C:0402-TIGHT, B.Cu at (95.3, 84.7)
- added R41: 150k, SparkFun ESP32 Thing Plus C:0402-TIGHT, B.Cu at (113.5, 70.4)
- added R42: 150k, SparkFun ESP32 Thing Plus C:0402-TIGHT, B.Cu at (113.5, 69.4)
- added R43: 150k, SparkFun ESP32 Thing Plus C:0402-TIGHT, B.Cu at (113.5, 68.4)
- added R44: 150k, SparkFun ESP32 Thing Plus C:0402-TIGHT, B.Cu at (113.5, 67.4)
- added R45: 150k, SparkFun ESP32 Thing Plus C:0402-TIGHT, B.Cu at (113.5, 65.4)
- added R46: 150k, SparkFun ESP32 Thing Plus C:0402-TIGHT, B.Cu at (113.5, 64.4)
- added R47: 150k, SparkFun ESP32 Thing Plus C:0402-TIGHT, B.Cu at (113.5, 63.4)
- added R48: 150k, SparkFun ESP32 Thing Plus C:0402-TIGHT, B.Cu at (113.5, 62.4)
- added R49: 150k, SparkFun ESP32 Thing Plus C:0402-TIGHT, B.Cu at (113.5, 60.4)
- added R50: 150k, SparkFun ESP32 Thing Plus C:0402-TIGHT, B.Cu at (113.5, 59.4)
- added R51: 150k, SparkFun ESP32 Thing Plus C:0402-TIGHT, B.Cu at (113.5, 57.4)
- added R52: 150k, SparkFun ESP32 Thing Plus C:0402-TIGHT, B.Cu at (113.5, 56.4)
- added R53: 150k, SparkFun ESP32 Thing Plus C:0402-TIGHT, B.Cu at (113.5, 55.4)
- added R54: 150k, SparkFun ESP32 Thing Plus C:0402-TIGHT, B.Cu at (113.5, 54.4)
- added R55: 150k, SparkFun ESP32 Thing Plus C:0402-TIGHT, B.Cu at (113.5, 53.4)
- added R56: 150k, SparkFun ESP32 Thing Plus C:0402-TIGHT, B.Cu at (113.5, 52.4)
- added R57: 10k, SparkFun ESP32 Thing Plus C:0402-TIGHT, B.Cu at (99.3, 70.2)
- added R58: 1k, SparkFun ESP32 Thing Plus C:0402-TIGHT, B.Cu at (107.0, 84.7)
- added R59: 2.0k, SparkFun ESP32 Thing Plus C:0402-TIGHT, B.Cu at (106.5, 78.6)
- added R60: 5.1k, SparkFun ESP32 Thing Plus C:0402-TIGHT, B.Cu at (103.3, 77.5)
- added R61: 5.1k, SparkFun ESP32 Thing Plus C:0402-TIGHT, B.Cu at (98.4, 77.6)
- added R62: 1k, SparkFun ESP32 Thing Plus C:0402-TIGHT, F.Cu at (92.9, 69.1)
- added S3: RES, Switches:TACTILE_SWITCH_SMD_2.8X1.9MM, F.Cu at (109.3, 74.1)
- added S4: B, Switches:TACTILE_SWITCH_SMD_2.8X1.9MM, F.Cu at (109.3, 70.4)
- added SW2: ON OFF, Button_Switch_SMD:SW_SPDT_k3-1295, B.Cu at (101.1, 84.1)
- added U12: , SparkFun ESP32 Thing Plus C:SOT23-5, B.Cu at (99.5, 81.0)
- added U13: >VALUE, SparkFun ESP32 Thing Plus C:ESP-WROOM-32-NARROW, F.Cu at (101.1, 56.8)
- added U14: MCP73831, SparkFun ESP32 Thing Plus C:SOT23-5, F.Cu at (107.6, 80.1)
- added U15: ADS1115IDGS, Package_SO:TSSOP-10_3x3mm_P0.5mm, B.Cu at (117.4, 71.9)
- added U16: ADS1115IDGS, Package_SO:TSSOP-10_3x3mm_P0.5mm, B.Cu at (117.4, 65.6)
- added U17: ADS1115IDGS, Package_SO:TSSOP-10_3x3mm_P0.5mm, B.Cu at (117.4, 59.3)
- added U18: ADS1115IDGS, Package_SO:TSSOP-10_3x3mm_P0.5mm, B.Cu at (117.4, 53.0)
- added U19: CH340C, PCM_Package_SO_AKL:SOIC-16_3.9x9.9mm_P1.27mm, F.Cu at (102.9, 73.1)
- added U20: MAX17048, SparkFun ESP32 Thing Plus C:DFN-8, B.Cu at (109.2, 78.6)
- D5: value BLUE -> S4 3A/10V/280mV; footprint SparkFun ESP32 Thing Plus C:LED-0603 -> SparkFun ESP32 Thing Plus C:SOD-323; moved to B.Cu
- R32: value 5.1k -> 10k
- R33: value 5.1k -> 4k7
- R34: value 1k -> 10k; moved to B.Cu
- U11: value MAX17048 -> ADXL345; footprint SparkFun ESP32 Thing Plus C:DFN-8 -> Package_LGA:LGA-14_3x5mm_P0.8mm_LayoutBorder1x6y
- moved R33 17.0 mm to (101.1, 61.2)
- moved U11 16.3 mm to (101.1, 64.4)
- moved R34 12.3 mm to (96.3, 80.9)
- moved D5 10.3 mm to (100.2, 77.9), turned to -90 degrees
- moved R32 2.47 mm to (101.4, 78.4), turned to -90 degrees
- moved REF** 2.35 mm to (93.3, 79.1), turned to 0 degrees
- moved JP4 0.91 mm to (107.1, 82.8)
- moved JP3 0.88 mm to (95.2, 82.8)
- moved G*** 0.55 mm to (115.8, 80.9)
- moved G*** 0.41 mm to (115.8, 45.8)
- moved mouse-bite-1mm-slot 0.40 mm to (115.9, 76.1)
- moved G*** 0.39 mm to (105.7, 46.2)
- moved mouse-bite-emm-slot 0.30 mm to (110.8, 80.9)
- renumbered JP1 to JP3, JP2 to JP4
Connections:
- D5 pad A: Net-(D5-PadA) -> V_USB
- D5 pad C: GND -> VIN
- R32 pad 2: Net-(J2-CC2) -> V_USB
- R33 pad 1: GND -> Net-(U11-SDO/ADDR)
- R33 pad 2: Net-(J2-CC1) -> GND
- R34 pad 1: /GPIO_13/ADC2_4/LED -> VIN
- R34 pad 2: Net-(D5-PadA) -> /EN
- REF** pad 1: V_BATT -> /V
- U11 pad 1: GND -> 3.3V
- U11 pad 2: V_BATT -> GND
- U11 pad 3: V_BATT -> unconnected-(U11-RES-Pad3)
- U11 pad 5: unconnected-(U11-~{ALRT}-Pad5) -> GND
- U11 pad 6: GND -> 3.3V
- U11 pad 7: /GPIO_22/SCL -> Net-(U11-~{CS})
- U11 pad 8: /GPIO_21/SDA -> unconnected-(U11-INT1-Pad8)
- U11 pad 9: GND -> unconnected-(U11-INT2-Pad9)
Routing:
- net GND: track 323.8 -> 704.5 mm, vias 90 -> 85
- net 3.3V: track 258.4 -> 352.6 mm, vias 24 -> 19
- net /V: track 0.00 -> 68.9 mm, vias 0 -> 9
- net V_BATT: track 94.5 -> 46.2 mm, vias 11 -> 6
- net V_USB: track 47.3 -> 75.8 mm, vias 6 -> 8
- net /A6: track 29.2 -> 12.1 mm
- net /A5: track 24.7 -> 9.83 mm
- net /GPIO_22/SCL: track 114.8 -> 126.9 mm, vias 7 -> 8
- net /A15: track 10.5 -> 22.0 mm
- net VIN: track 8.86 -> 18.4 mm
- net /A2: track 20.7 -> 11.1 mm
- net /A9: track 16.9 -> 7.77 mm
- net /~{RESET}: track 56.2 -> 47.9 mm
- net /GPIO_21/SDA: track 121.8 -> 129.3 mm, vias 12 -> 11
- net /A10: track 23.4 -> 17.1 mm
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- added copper zone on B.Cu, net /V
- added copper zone on F.Cu, net /V
- removed copper zone on B.Cu, net V_BATT
- removed copper zone on F.Cu, net V_BATT
Other:
- outline, holes or cut-outs redrawn

Commit message: .
Parts:
- S3: renamed from S4; value B -> Boot
- S4: renamed from S3; value RES -> Reset
- SW2: value ON OFF -> ON/OFF
Connections:
- U12 pad 4: GND -> unconnected-(U12-NC-Pad4)
