File: ESP32-DEVKIT-S rev1/panelization/panelization.kicad_pcb (KiCad board)
At the start: 2 copper layers, 57.9 x 42.5 mm, 179 parts, among them J1 JST_2MM_MALE, J10 QWIIC_RIGHT_ANGLE, J11 Conn_01x20, J12 Conn_01x20, J13 QWIIC_RIGHT_ANGLE, J14 Conn_01x20, J2 USB_C_2-LAYER_PADS, J3 Conn_01x20, J4 QWIIC_RIGHT_ANGLE, J5 Conn_01x20, J6 Conn_01x20, J7 QWIIC_RIGHT_ANGLE, J8 JST_2MM_MALE, J9 USB_C_2-LAYER_PADS, Q1 DMG2305UX 20V/4.2A/52mΩ/1.4W, Q2 MBT3904DW1T1, Q3 DMG2305UX 20V/4.2A/52mΩ/1.4W, Q4 MBT3904DW1T1, SW1 ON OFF, SW2 ON OFF, U1 ADXL345, U11 ADXL345, U11 MAX17048, U13 >VALUE, U14 MCP73831, U15 ADS1115IDGS, U16 ADS1115IDGS, U17 ADS1115IDGS, U18 ADS1115IDGS, U19 CH340C, U20 MAX17048, U3 >VALUE, U4 MCP73831, U5 ADS1115IDGS, U6 ADS1115IDGS, U7 ADS1115IDGS, U8 ADS1115IDGS, U9 CH340C

Commit message: .
Parts:
- removed the >NAME at (130.6, 36.6)
- removed the >NAME at (130.6, 49.1)
- removed the >NAME at (130.6, 42.8)
- removed the >NAME at (130.6, 30.3)
- removed the ? at (106.4, 61.2)
- removed the ? at (122.3, 61.2)
- removed the G*** at (129.0, 23.1)
- removed the G*** at (129.0, 58.1)
- removed the G*** at (118.9, 23.4)
- removed the mouse-bite-emm-slot at (124.0, 27.9)
- removed the mouse-bite-emm-slot at (124.0, 51.6)
- removed the mouse-bite-emm-slot at (124.0, 58.1)
- removed the mouse-bite-emm-slot at (124.0, 39.7)
- added >NAME: >VALUE, Silicon-Standard:QFN-10-RSE, B.Cu at (130.7, 30.3)
- added >NAME: >VALUE, Silicon-Standard:QFN-10-RSE, B.Cu at (130.7, 42.8)
- added >NAME: >VALUE, Silicon-Standard:QFN-10-RSE, B.Cu at (130.7, 36.6)
- added >NAME: >VALUE, Silicon-Standard:QFN-10-RSE, B.Cu at (130.7, 49.1)
- added ?: , , F.Cu at (122.4, 61.2)
- added ?: , , F.Cu at (106.4, 61.2)
- added G***: LOGO, logo:Hasatio_logo_mini, B.Cu at (129.1, 23.1)
- added G***: LOGO, logo:Hasatio_logo_mini, B.Cu at (118.9, 23.4)
- added G***: LOGO, logo:Hasatio_logo_mini, B.Cu at (129.1, 58.1)
- added mouse-bite-emm-slot: VAL**, Panelization:mouse-bite-1mm 2, F.Cu at (124.0, 58.1)
- added mouse-bite-emm-slot: VAL**, Panelization:mouse-bite-1mm 2, F.Cu at (124.0, 51.6)
- added mouse-bite-emm-slot: VAL**, Panelization:mouse-bite-1mm 2, F.Cu at (124.0, 39.7)
- added mouse-bite-emm-slot: VAL**, Panelization:mouse-bite-1mm 2, F.Cu at (124.0, 27.9)
- S1: value B -> Boot
- S2: value RES -> Reset
- S3: value RES -> Boot
- S4: value B -> Reset
- SW1, SW2: value ON OFF -> ON/OFF
- moved S3 3.66 mm to (122.6, 47.7), turned to 90 degrees
- moved S4 3.66 mm to (122.6, 51.3), turned to -90 degrees
- moved C18 0.05 mm to (114.7, 47.9)
- moved C28 0.05 mm to (119.0, 58.3)
- moved D5 0.05 mm to (113.4, 55.2)
- moved J14 0.05 mm to (118.9, 40.6)
- moved J8 0.05 mm to (130.6, 58.1)
- moved R32 0.05 mm to (114.7, 55.6)
- moved R33 0.05 mm to (114.3, 38.5)
- moved R61 0.05 mm to (111.6, 54.8)
- moved U15 0.05 mm to (130.7, 49.1)
- moved U16 0.05 mm to (130.7, 42.8)
- moved U17 0.05 mm to (130.7, 36.6)
- moved U18 0.05 mm to (130.7, 30.3)
- renumbered C14 to C13, C13 to C14, J7 to J3, J6 to J4, J3 to J5, J4 to J6, J5 to J7, U11 to U10
Connections:
- net Board_0-Net-(D5-PadA) renamed Board_0-Net-(D4-PadA)
- net Board_0-unconnected-(J6-Pin_10-Pad10) renamed Board_0-unconnected-(J4-Pin_10-Pad10)
- net Board_0-unconnected-(J6-Pin_20-Pad20) renamed Board_0-unconnected-(J4-Pin_20-Pad20)
- net Board_0-unconnected-(U11-~{ALRT}-Pad5) renamed Board_0-unconnected-(U10-~{ALRT}-Pad5)
- S3 pad 1: Board_1-/~{RESET} -> Board_1-/GPIO_0/ADC2_1/QPWR
- S3 pad 3: Board_1-/~{RESET} -> Board_1-/GPIO_0/ADC2_1/QPWR
- S4 pad 1: Board_1-/GPIO_0/ADC2_1/QPWR -> Board_1-/~{RESET}
- S4 pad 3: Board_1-/GPIO_0/ADC2_1/QPWR -> Board_1-/~{RESET}
- U12 pad 4: Board_1-GND -> Board_1-unconnected-(U12-NC-Pad4)
- U2 pad 4: Board_0-VIN -> Board_0-unconnected-(U2-NC-Pad4)
Routing:
- net Board_0-GND: track 672.7 -> 681.5 mm, vias 87 -> 88
- net Board_0-/GPIO_22/SCL: track 140.1 -> 143.3 mm
- net Board_0-3.3V: track 342.0 -> 344.1 mm
- net Board_0-V_USB: track 33.6 -> 32.7 mm
- net Board_0-/~{RESET}: track 48.0 -> 48.6 mm
Other:
- board size 57.9 x 42.5 mm -> 58 x 42.5 mm
- board text removed: "V-CUT"
