File: Rev1/panelization/panelization.kicad_sch (KiCad schematic)
At the start: 0 parts

Commit message: .
Other:
- sheet ESP32-DEVKIT-S-ch340 renamed R
- sheet ESP32-DEVKIT-S-ch340-mirror renamed L
- sheet L: file ../ESP32-DEVKIT-S-mirror/ESP32-DEVKIT-S-ch340-mirror.kicad_sch -> F:/OneDrive/proje/git/Hasatio/esp32DevKitS/Rev1/L/L.kicad_sch
- sheet R: file ../ESP32-DEVKIT-S/ESP32-DEVKIT-S-ch340.kicad_sch -> F:/OneDrive/proje/git/Hasatio/esp32DevKitS/Rev1/R/R.kicad_sch
Changed lines of the file:
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@@
     (stroke (width 0.1524) (type solid))
     (fill (color 0 0 0 0.0000))
-    (property "Sheetname" "ESP32-DEVKIT-S-ch340-mirror" (at 120.65 53.8984 0)
+    (property "Sheetname" "L" (at 120.65 53.8984 0)
       (effects (font (size 1.27 1.27)) (justify left bottom))
     )
-    (property "Sheetfile" "../ESP32-DEVKIT-S-mirror/ESP32-DEVKIT-S-ch340-mirror.kicad_sch" (at 120.65 59.0046 0)
+    (property "Sheetfile" "F:/OneDrive/proje/git/Hasatio/esp32DevKitS/Rev1/L/L.kicad_sch" (at 120.65 59.0046 0)
       (effects (font (size 1.27 1.27)) (justify left top))
     )
@@
     (stroke (width 0.1524) (type solid))
     (fill (color 0 0 0 0.0000))
-    (property "Sheetname" "ESP32-DEVKIT-S-ch340" (at 67.31 53.8984 0)
+    (property "Sheetname" "R" (at 67.31 53.8984 0)
       (effects (font (size 1.27 1.27)) (justify left bottom))
     )
-    (property "Sheetfile" "../ESP32-DEVKIT-S/ESP32-DEVKIT-S-ch340.kicad_sch" (at 67.31 59.0046 0)
+    (property "Sheetfile" "F:/OneDrive/proje/git/Hasatio/esp32DevKitS/Rev1/R/R.kicad_sch" (at 67.31 59.0046 0)
       (effects (font (size 1.27 1.27)) (justify left top))
     )
