File: Rev0/Rev0.kicad_sch (KiCad schematic)
At the start: 75 parts, among them J1 JST_2MM_MALE, J2 USB_C_2-LAYER_PADS, J3 Conn_01x20, J4 QWIIC_RIGHT_ANGLE, J5 Conn_01x20, J6 Conn_01x20, J7 QWIIC_RIGHT_ANGLE, Q1 DMG2305UX 20V/4.2A/52mΩ/1.4W, Q2 MBT3904DW1T1, U1 ADXL345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

Commit message: .
Other:
- company: hasatio -> HASATIO
- title: posture -> ESP32-DEVKIT-S
