File: Rev1/L/L.kicad_sch (KiCad schematic)
At the start: 75 parts, among them J10 QWIIC_RIGHT_ANGLE, J11 Conn_01x20, J12 Conn_01x20, J13 QWIIC_RIGHT_ANGLE, J14 Conn_01x20, J8 JST_2MM_MALE, J9 USB_C_2-LAYER_PADS, Q3 DMG2305UX 20V/4.2A/52mΩ/1.4W, Q4 MBT3904DW1T1, SW2 ON/OFF, U11 ADXL345, U13 >VALUE, U14 MCP73831, U15 ADS1115IDGS, U16 ADS1115IDGS, U17 ADS1115IDGS, U18 ADS1115IDGS, U19 CH340C, U20 MAX17048

Commit message: .
Parts:
- added C15, C16, C17, C22, C23, C24, C25, C27: 1.0uF, SparkFun ESP32 Thing Plus C:0402-TIGHT, symbol SparkFun ESP32 Thing Plus C-eagle-import:1.0UF-0402T-16V-10%
- added C18, C19: 10uF, SparkFun ESP32 Thing Plus C:0402-TIGHT, symbol SparkFun ESP32 Thing Plus C-eagle-import:10UF-0402T-6.3V-20%
- added C20: 4.7uF, SparkFun ESP32 Thing Plus C:0402-TIGHT, symbol SparkFun ESP32 Thing Plus C-eagle-import:4.7UF-0603-35V-(20%)
- added C21: 4.7uF, SparkFun ESP32 Thing Plus C:0402-TIGHT, symbol SparkFun ESP32 Thing Plus C-eagle-import:4.7UF-0402_TIGHT-6.3V-20%-X5R
- added C26: 0.1uF, SparkFun ESP32 Thing Plus C:0402-TIGHT, symbol SparkFun ESP32 Thing Plus C-eagle-import:0.1UF-0402T-6.3V-10%-X7R
- added C28: 0.1uF, SparkFun ESP32 Thing Plus C:0402-TIGHT, symbol SparkFun ESP32 Thing Plus C-eagle-import:0.1UF-0402T-16V-10%
- added D5: S4 3A/10V/280mV, SparkFun ESP32 Thing Plus C:SOD-323, symbol SparkFun ESP32 Thing Plus C-eagle-import:DIODE-SCHOTTKY-BAT60A
- added D6: RED, SparkFun ESP32 Thing Plus C:LED-0603, symbol SparkFun ESP32 Thing Plus C-eagle-import:LED-RED0603
- added D7: Yellow, SparkFun ESP32 Thing Plus C:LED-0603, symbol SparkFun ESP32 Thing Plus C-eagle-import:LED-YELLOW0603
- added D8: BLUE, SparkFun ESP32 Thing Plus C:LED-0603, symbol SparkFun ESP32 Thing Plus C-eagle-import:LED-BLUE0603
- added J10, J13: QWIIC_RIGHT_ANGLE, SparkFun ESP32 Thing Plus C:JST04_1MM_RA, symbol SparkFun ESP32 Thing Plus C-eagle-import:QWIIC_CONNECTORJS-1MM
- added J11, J12, J14: Conn_01x20, Connector_FFC-FPC:Molex_200528-0200_1x20-1MP_P1.00mm_Horizontal, symbol Connector_Generic:Conn_01x20
- added J8: JST_2MM_MALE, SparkFun ESP32 Thing Plus C:JST-2-SMD, symbol SparkFun ESP32 Thing Plus C-eagle-import:JST_2MM_MALE
- added J9: USB_C_2-LAYER_PADS, SparkFun ESP32 Thing Plus C:USB-C-16P-2LAYER-PADS, symbol SparkFun ESP32 Thing Plus C-eagle-import:USB_C_2-LAYER_PADS
- added JP3, JP4: JUMPER-SMT_2_NC_TRACE_SILK, SparkFun ESP32 Thing Plus C:SMT-JUMPER_2_NC_TRACE_SILK, symbol SparkFun ESP32 Thing Plus C-eagle-import:JUMPER-SMT_2_NC_TRACE_SILK
- added LOGO3: QWIIC_LOGO_4MM, SparkFun ESP32 Thing Plus C:QWIIC_4MM, symbol SparkFun ESP32 Thing Plus C-eagle-import:QWIIC_LOGO_4MM
- added LOGO4: OSHW-LOGOMINI, SparkFun ESP32 Thing Plus C:OSHW-LOGO-MINI, symbol SparkFun ESP32 Thing Plus C-eagle-import:OSHW-LOGOMINI
- added Q3: DMG2305UX 20V/4.2A/52mΩ/1.4W, SparkFun ESP32 Thing Plus C:SOT23-3, symbol SparkFun ESP32 Thing Plus C-eagle-import:MOSFET_PCH-DMG2305UX-7
- added Q4: MBT3904DW1T1, SparkFun ESP32 Thing Plus C:SC70-6, symbol SparkFun ESP32 Thing Plus C-eagle-import:TRANS_NPN_DUAL-MBT3904DW1T1
- added R32, R34, R35, R38, R39, R57: 10k, SparkFun ESP32 Thing Plus C:0402-TIGHT, symbol SparkFun ESP32 Thing Plus C-eagle-import:10KOHM-0402T-1/16W-1%
- added R33, R36, R37: 4k7, SparkFun ESP32 Thing Plus C:0402-TIGHT, symbol SparkFun ESP32 Thing Plus C-eagle-import:10KOHM-0402T-1/16W-1%
- added R40, R58, R62: 1k, SparkFun ESP32 Thing Plus C:0402-TIGHT, symbol SparkFun ESP32 Thing Plus C-eagle-import:1KOHM-0402T-1/16W-1%
- added R41, R42, R43, R44, R45, R46, R47, R48, R49, R50, R51, R52, R53, R54, R55, R56: 150k, SparkFun ESP32 Thing Plus C:0402-TIGHT, symbol SparkFun ESP32 Thing Plus C-eagle-import:10KOHM-0402T-1/16W-1%
- added R59: 2.0k, SparkFun ESP32 Thing Plus C:0402-TIGHT, symbol SparkFun ESP32 Thing Plus C-eagle-import:2.0KOHM-0603-1/10W-5%
- added R60, R61: 5.1k, SparkFun ESP32 Thing Plus C:0402-TIGHT, symbol SparkFun ESP32 Thing Plus C-eagle-import:5.1KOHM-0402T-1/16W-1%
- added S3: Boot, Switches:TACTILE_SWITCH_SMD_2.8X1.9MM, symbol Switch:SW_Push_Dual
- added S4: Reset, Switches:TACTILE_SWITCH_SMD_2.8X1.9MM, symbol Switch:SW_Push_Dual
- added SW2: ON/OFF, Button_Switch_SMD:SW_SPDT_k3-1295, symbol Switch:SW_SPDT
- added U11: ADXL345, Package_LGA:LGA-14_3x5mm_P0.8mm_LayoutBorder1x6y, symbol Sensor_Motion:ADXL343
- added U12: (no value), SparkFun ESP32 Thing Plus C:SOT23-5, symbol SparkFun ESP32 Thing Plus C-eagle-import:V_REG_AP2112K-3.3V
- added U13: >VALUE, SparkFun ESP32 Thing Plus C:ESP-WROOM-32-NARROW, symbol RF_Module:ESP32-WROOM-32
- added U14: MCP73831, SparkFun ESP32 Thing Plus C:SOT23-5, symbol SparkFun ESP32 Thing Plus C-eagle-import:MCP73831
- added U15, U16, U17, U18: ADS1115IDGS, Package_SO:TSSOP-10_3x3mm_P0.5mm, symbol Analog_ADC:ADS1115IDGS
- added U19: CH340C, PCM_Package_SO_AKL:SOIC-16_3.9x9.9mm_P1.27mm, symbol Interface_USB:CH340C
- added U20: MAX17048, SparkFun ESP32 Thing Plus C:DFN-8, symbol SparkFun ESP32 Thing Plus C-eagle-import:MAX17048DFN8
Connections:
- net 3.3V: now also C16.1, C17.1, C18.1, C19.1, C22.1, C23.1, C24.1, C25.1, C26.1, C27.1, J10.2, J12.19 (Pin_19), J12.2 (Pin_2), J13.2, J14.19 (Pin_19), J14.2 (Pin_2), JP3.2, R35.1, R36.1, R37.1, R41.2, R42.2, R43.2, R44.2, R45.2, R46.2, R47.2, R48.2, R49.1, R50.1, R51.1, R52.1, R53.1, R54.1, R55.1, R56.1, R57.1, U11.1 (Vdd_I/O), U11.6 (Vs), U12.5 (OUT), U13.2 (VDD), U15.8 (VDD), U16.1 (ADDR), U16.8 (VDD), U17.8 (VDD), U18.8 (VDD), U19.16 (VCC), U19.4 (V3)
- net A1: now also J11.2 (Pin_2), R41.1, U15.4 (AIN0)
- net A10: now also J11.13 (Pin_13), R50.2, U17.5 (AIN1)
- net A11: now also J11.15 (Pin_15), R51.2, U17.6 (AIN2)
- net A12: now also J11.16 (Pin_16), R52.2, U17.7 (AIN3)
- net A13: now also J11.17 (Pin_17), R53.2, U18.4 (AIN0)
- net A14: now also J11.18 (Pin_18), R54.2, U18.5 (AIN1)
- net A15: now also J11.19 (Pin_19), R55.2, U18.6 (AIN2)
- net A16: now also J11.20 (Pin_20), R56.2, U18.7 (AIN3)
- net A2: now also J11.3 (Pin_3), R42.1, U15.5 (AIN1)
- net A3: now also J11.4 (Pin_4), R43.1, U15.6 (AIN2)
- net A4: now also J11.5 (Pin_5), R44.1, U15.7 (AIN3)
- net A5: now also J11.7 (Pin_7), R45.1, U16.4 (AIN0)
- net A6: now also J11.8 (Pin_8), R46.1, U16.5 (AIN1)
- net A7: now also J11.9 (Pin_9), R47.1, U16.6 (AIN2)
- net A8: now also J11.10 (Pin_10), R48.1, U16.7 (AIN3)
- net A9: now also J11.12 (Pin_12), R49.2, U17.4 (AIN0)
- net CH340-DTR: now also Q4.1 (E), R38.1, U19.13 (~{DTR})
- net CH340-RTS: now also Q4.4 (E), R39.1, U19.14 (~{RTS})
- net D+: now also J9.A6 (D+), J9.B6 (D+), U19.5 (UD+)
- net D-: now also J9.A7 (D-), J9.B7 (D-), U19.6 (UD-)
- net EN: now also R34.2, U12.3 (EN)
- net GND: now also C15.2, C16.2, C17.2, C18.2, C19.2, C20.2, C21.2, C22.2, C23.2, C24.2, C25.2, C26.2, C27.2, C28.2, D6.C, D8.C, J10.1, J11.14 (Pin_14), J11.6 (Pin_6), J12.1 (Pin_1), J12.20 (Pin_20), J13.1, J14.1 (Pin_1), J14.20 (Pin_20), J8.1 (-), J9.GND, J9.GND2 (GND), J9.SHLD1 (SHLD), J9.SHLD2 (SHLD), J9.SHLD3 (SHLD), J9.SHLD4 (SHLD), R32.1, R33.2, R59.1, R60.1, R61.1, S3.2, S3.4, S4.2, S4.4, SW2.GND, U11.2 (GND), U11.4 (GND), U11.5 (GND), U12.2 (GND), U13.1 (GND), U13.15 (GND), U13.38 (GND), U13.39 (GND), U14.2 (VSS), U15.1 (ADDR), U15.3 (GND), U16.3 (GND), U17.3 (GND), U18.3 (GND), U19.1 (GND), U20.1 (CTG), U20.4 (GND), U20.6 (QSTRT), U20.9 (GND)
- net GPIO_0/ADC2_1/QPWR: now also J14.14 (Pin_14), Q4.6 (C), S3.1, S3.3, U13.25 (IO0)
- net GPIO_1/TX: now also J14.5 (Pin_5), U13.35 (TXD0/IO1)
- net GPIO_10/SWP: now also J12.5 (Pin_5), U13.18 (SWP/SD3)
- net GPIO_11/SCS: now also J12.4 (Pin_4), U13.19 (SCS/CMD)
- net GPIO_12/ADC2_5: now also J12.8 (Pin_8), U13.14 (IO12)
- net GPIO_13/ADC2_4/LED: now also J12.7 (Pin_7), R62.1, U13.16 (IO13)
- net GPIO_14/ADC2_6: now also J12.9 (Pin_9), U13.13 (IO14)
- net GPIO_15/ADC2_3: now also J14.16 (Pin_16), U13.23 (IO15)
- net GPIO_16/RX: now also J14.12 (Pin_12), U13.27 (IO16)
- net GPIO_17/TX: now also J14.11 (Pin_11), U13.28 (IO17)
- net GPIO_18/SCK: now also J14.9 (Pin_9), U13.30 (IO18)
- net GPIO_19/CIPO: now also J14.8 (Pin_8), U13.31 (IO19)
- net GPIO_1/TX: now also U19.3 (RXD)
- net GPIO_2/ADC2_2: now also J14.15 (Pin_15), U13.24 (IO2)
- net GPIO_21/SDA: now also J10.3, J13.3, J14.7 (Pin_7), R37.2, U11.13 (SDA/SDI/SDIO), U13.33 (IO21), U15.9 (SDA), U16.9 (SDA), U17.1 (ADDR), U17.9 (SDA), U18.9 (SDA), U20.8 (SDA)
- net GPIO_22/SCL: now also J10.4, J13.4, J14.4 (Pin_4), R36.2, U11.14 (SCL/SCLK), U13.36 (IO22), U15.10 (SCL), U16.10 (SCL), U17.10 (SCL), U18.1 (ADDR), U18.10 (SCL), U20.7 (SCL)
- net GPIO_23/COPI: now also J14.3 (Pin_3), U13.37 (IO23)
- net GPIO_25/ADC2_8: now also J12.12 (Pin_12), U13.10 (IO25)
- net GPIO_26/ADC2_9: now also J12.11 (Pin_11), U13.11 (IO26)
- net GPIO_27/ADC2_7: now also J12.10 (Pin_10), U13.12 (IO27)
- net GPIO_3/RX: now also J14.6 (Pin_6), U13.34 (RXD0/IO3)
- net GPIO_32/ADC1_4: now also J12.14 (Pin_14), U13.8 (IO32)
- net GPIO_33/ADC1_5: now also J12.13 (Pin_13), U13.9 (IO33)
- net GPIO_34/ADC1_6: now also J12.16 (Pin_16), U13.6 (IO34)
- net GPIO_35/ADC1_7: now also J12.15 (Pin_15), U13.7 (IO35)
- net GPIO_36/ADC1_0: now also J12.18 (Pin_18), U13.4 (SENSOR_VP)
- net GPIO_39/ADC1_3: now also J12.17 (Pin_17), U13.5 (SENSOR_VN)
- net GPIO_3/RX: now also U19.2 (TXD)
- net GPIO_4/ADC2_0: now also J14.13 (Pin_13), U13.26 (IO4)
- net GPIO_5/SD_CS: now also J14.10 (Pin_10), U13.29 (IO5)
- net GPIO_6/SCK: now also J12.3 (Pin_3), U13.20 (SCK/CLK)
- net GPIO_7/SDO: now also J14.18 (Pin_18), U13.21 (SDO/SD0)
- net GPIO_8/SDI: now also J14.17 (Pin_17), U13.22 (SDI/SD1)
- net GPIO_9/SHD: now also J12.6 (Pin_6), U13.17 (SHD/SD2)
- net V: now also J8.2 (+), SW2.2 (B)
- net VIN: now also C15.1, D5.C, Q3.2 (S), R34.1, U12.1 (IN)
- net V_BATT: now also C21.1, C28.1, Q3.3 (D), SW2.1 (A), U14.3 (VBAT), U20.2 (CELL), U20.3 (VDD)
- net V_USB: now also C20.1, D5.A, J9.VBUS1 (VBUS), J9.VBUS2 (VBUS), JP4.2, Q3.1 (G), R32.2, U14.4 (VIN)
- net ~{RESET}: now also Q4.3 (C), R57.2, S4.1, S4.3, U13.3 (EN)
- net at D6.A, R40.2: now also D6.A, R40.2
- net at JP3.1, R40.1: now also JP3.1, R40.1
- net at Q4.2 (B), R39.2: now also Q4.2 (B), R39.2
- net at Q4.5 (B), R38.2: now also Q4.5 (B), R38.2
- net at R35.2, U11.7 (~{CS}): now also R35.2, U11.7 (~{CS})
- net at D7.A, R58.2: now also D7.A, R58.2
- net at D7.C, U14.1 (STAT): now also D7.C, U14.1 (STAT)
- net at R59.2, U14.5 (PROG): now also R59.2, U14.5 (PROG)
- net at J8.NC1 (PAD1): now also J8.NC1 (PAD1)
- net at J8.NC2 (PAD2): now also J8.NC2 (PAD2)
- net at U19.10 (~{DSR}): now also U19.10 (~{DSR})
- net at U19.11 (~{RI}): now also U19.11 (~{RI})
- net at U19.12 (~{DCD}): now also U19.12 (~{DCD})
- net at U19.15 (R232): now also U19.15 (R232)
- net at U19.7 (NC): now also U19.7 (NC)
- net at U19.8 (NC): now also U19.8 (NC)
- net at U19.9 (~{CTS}): now also U19.9 (~{CTS})
- net at JP4.1, R58.1: now also JP4.1, R58.1
- net at SW2.3 (C): now also SW2.3 (C)
- net at J9.A5 (CC1), R61.2: now also J9.A5 (CC1), R61.2
- net at D8.A, R62.2: now also D8.A, R62.2
- net at U12.4 (NC): now also U12.4 (NC)
- net at U15.2 (ALERT/RDY): now also U15.2 (ALERT/RDY)
- net at J11.1 (Pin_1): now also J11.1 (Pin_1)
- net at J11.11 (Pin_11): now also J11.11 (Pin_11)
- net at J9.B5 (CC2), R60.2: now also J9.B5 (CC2), R60.2
- net at U13.32 (NC): now also U13.32 (NC)
- net at U16.2 (ALERT/RDY): now also U16.2 (ALERT/RDY)
- net at U18.2 (ALERT/RDY): now also U18.2 (ALERT/RDY)
- net at R33.1, U11.12 (SDO/ADDR): now also R33.1, U11.12 (SDO/ADDR)
- net at U17.2 (ALERT/RDY): now also U17.2 (ALERT/RDY)
- net at U11.10 (NC): now also U11.10 (NC)
- net at U11.11 (RES): now also U11.11 (RES)
- net at U11.3 (RES): now also U11.3 (RES)
- net at U11.8 (INT1): now also U11.8 (INT1)
- net at U11.9 (INT2): now also U11.9 (INT2)
- net at U20.5 (~{ALRT}): now also U20.5 (~{ALRT})

Commit message: .
Other:
- company: hasatio -> HASATIO
- title: posture -> ESP32-DEVKIT-S
Changed lines of the file:
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@@
   (paper "User" 451.815 299.39)
   (title_block
-    (title "posture")
-    (date "2023-02-28")
-    (rev "0")
-    (company "hasatio")
+    (title "ESP32-DEVKIT-S")
+    (rev "1")
+    (company "HASATIO")
   )
   (junction (at 53.34 256.54) (diameter 0) (color 0 0 0 0)
