File: Rev1/R/R.kicad_sch (KiCad schematic)
At the start: 75 parts, among them J1 JST_2MM_MALE, J2 USB_C_2-LAYER_PADS, J3 QWIIC_RIGHT_ANGLE, J4 Conn_01x20, J5 Conn_01x20, J6 QWIIC_RIGHT_ANGLE, J7 Conn_01x20, Q1 DMG2305UX 20V/4.2A/52mΩ/1.4W, Q2 MBT3904DW1T1, SW1 ON/OFF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

Commit message: .
Other:
- company: hasatio -> HASATIO
- title: posture -> ESP32-DEVKIT-S
