File: Rev2/R/R.kicad_sch (KiCad schematic)
At the start: 75 parts, among them J1 JST_2MM_MALE, J2 USB_C_2-LAYER_PADS, J3 QWIIC_RIGHT_ANGLE, J4 Conn_01x20, J5 Conn_01x20, J6 QWIIC_RIGHT_ANGLE, J7 Conn_01x20, Q1 DMG2305UX 20V/4.2A/52mΩ/1.4W, Q2 MBT3904DW1T1, SW1 ON/OFF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

Commit message: .
Parts:
- removed C13: 1.0uF, SparkFun ESP32 Thing Plus C:0402-TIGHT, symbol SparkFun ESP32 Thing Plus C-eagle-import:1.0UF-0402T-16V-10%
- removed J3, J6: QWIIC_RIGHT_ANGLE, SparkFun ESP32 Thing Plus C:JST04_1MM_RA, symbol SparkFun ESP32 Thing Plus C-eagle-import:QWIIC_CONNECTORJS-1MM
- added C25: 0.1uF, SparkFun ESP32 Thing Plus C:0402-TIGHT, symbol SparkFun ESP32 Thing Plus C-eagle-import:1.0UF-0402T-16V-10%
- added C27: 1.0uF, SparkFun ESP32 Thing Plus C:0402-TIGHT, symbol SparkFun ESP32 Thing Plus C-eagle-import:1.0UF-0402T-16V-10%
- added J10 (x2): QWIIC_RIGHT_ANGLE, SparkFun ESP32 Thing Plus C:JST04_1MM_RA, symbol SparkFun ESP32 Thing Plus C-eagle-import:QWIIC_CONNECTORJS-1MM
- C10, C11, C2, C8, C9: value 1.0uF -> 0.1uF
Connections:
- net 3.3V: now also C25.1, C27.1, J10.2, J10.2
- net GND: now also C25.2, C27.2, J10.1, J10.1
- net GPIO_21/SDA: now also J10.3, J10.3
- net GPIO_22/SCL: now also J10.4, J10.4
Other:
- moved on the sheet: C10, C11, C8, C9

Commit message: .
Other:
- company: hasatio -> HASATIO
- title: posture -> ESP32-DEVKIT-S
Changed lines of the file:
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@@
   (paper "User" 451.815 299.39)
   (title_block
-    (title "posture")
-    (date "2023-02-28")
-    (rev "0")
-    (company "hasatio")
+    (title "ESP32-DEVKIT-S")
+    (rev "2")
+    (company "HASATIO")
   )
   (junction (at 88.9 160.02) (diameter 0) (color 0 0 0 0)
